File: cad/kicad/MotoRecoPico.kicad_sch (KiCad schematic)
At the start: 41 parts, among them J1 1-967658-1, J2 DM3AT-SF-PEJM5, J3 GT-502MGG-N, Q1 MMBT3904, Q2 ZXMP6A17E6Q, U2 MCP25625, U3 Pico 2, U4 AP63205WU-7, Y1 16MHz

Commit message: Add the v5 JLCPCB-assembly board variant (MRP_ASSY=jlc) with J4 direct-wire pads
Board and schematic are now the v5 build: all 37 machine-placed SMT parts on
the top face, the Pico soldered flush to the bottom face via castellations
(custom Pico2-SMD-Flush footprint), GPS off the board (wired straight to the
Pico), Q2 -> SI2309, Y1 -> 3225 SMD, chips 0603 to stay on HASL.

J4 adds five bare solder pads between J1 and the board edge on the Pico face
for wiring the vehicle loom directly: L H I G V (CANL, CANH, IGN, GND, +12V
upstream of F1) in the same left-to-right order as the J1 pins they tap, so
ses_import draws the five escapes straight from the J1 barrels on B.Cu with
no vias; dsn_export hides J4 and its lanes from the autorouter.

Freerouting is now 2.5.0: try_thermal's parser and -mp follow the new CLI,
xtal_check tolerates the fanout vias, and two new gates reject bad seeds
(plane_gate.py for In1 GND fragments, drc_detail.py prints what DRC hit).
jlc_top.py writes the top-face-only BOM/CPL pair for the assembly order, and
docs/datasheets holds the vendor PDFs behind the polarity check.

Co-Authored-By: Claude Fable 5 <noreply@anthropic.com>
Parts:
- removed J3: GT-502MGG-N, MotoRecoPico:GPS-5P-SMD-2.54, symbol Connector_Generic:Conn_01x05
- added J4: DIRECT-WIRE, MotoRecoPico:PAD-5P-DIRECT, symbol Connector_Generic:Conn_01x05
- C13: footprint Capacitor_SMD:C_0603_1608Metric -> Capacitor_SMD:C_0805_2012Metric
- C16: footprint Capacitor_SMD:C_0805_2012Metric -> Capacitor_SMD:C_0603_1608Metric
- C7, C8: value 22pF -> 12pF
- L1: footprint MotoRecoPico:L_4030_HandSolder -> Inductor_SMD:L_Abracon_ASPI-4030S
- Q2: value ZXMP6A17E6Q -> SI2309; footprint Package_TO_SOT_SMD:TSOT-23-6_HandSoldering -> Package_TO_SOT_SMD:SOT-23; symbol MotoRecoPico:ZXMP6A17E6Q -> Transistor_FET:Q_PMOS_GSD
- U3: footprint Module:RaspberryPi_Pico_Common_THT -> MotoRecoPico:Pico2-SMD-Flush
- U4: footprint Package_TO_SOT_SMD:TSOT-23-6_HandSoldering -> Package_TO_SOT_SMD:TSOT-23-6
- Y1: footprint Crystal:Crystal_HC49-4H_Vertical -> Crystal:Crystal_SMD_3225-4Pin_3.2x2.5mm; symbol Device:Crystal -> Device:Crystal_GND24
Connections:
- net CANH: now also J4.2 (Pin_2)
- net CANL: now also J4.1 (Pin_1)
- net GND: now also Y1.2 (G), Y1.4 (G), J4.4 (Pin_4)
- net IG_RAW: now also J4.3 (Pin_3)
- net V12_RAW: now reaches F1.1, J1.8 (Pin_8)
- net V12_RAW: now also J4.5 (Pin_5)
- net at C8.1, U2.8 (OSC2): now also Y1.3; no longer Y1.2
- net at C13.1, R1.2, R2.1: now also Q2.1 (G); no longer Q2.3 (G)
- net at C13.2, C2.1, D1.1 (K)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: now also Q2.2 (S); no longer Q2.4 (S)
- net GPS_PPS: no longer names the net of U3.9 (GPIO6)
- net GPS_RX: no longer names the net of U3.2 (GPIO1)
- net GPS_TX: no longer names the net of U3.1 (GPIO0)
- new net: C14.1, Q2.3 (D), U4.2 (EN), U4.3 (IN)
- no-connect marks 21 -> 24
Other:
- note added: "GPS module: 5 wires straight to the Pico (GP0/GP1/GP6 + 3V3/GND)"
- note added: "J4: direct-wire pads on the Pico face (V=12V I=IGN G=GND H=CANH L=CANL)"
- note removed: "GPS GT-502MGG-N"
- moved on the sheet: C13, R1, R2
